Commit message: 2024.12.30

File: ymbot_ocs2/ymbot_d_description/urdf/old.urdf (robot description, URDF)
Before this commit: robot ymbot_d_description, 34 links, 33 joints
Links:
- link Body_Link1: geometry collision mesh filename=package://ymbot_d_description/meshes/Body_Link1.STL; visual mesh filename=package://ymbot_d_description/meshes/Body_Link1.STL

Commit message: 2025.1.6

File: ymbot_ocs2/ymbot_d_description/urdf/old.urdf (robot description, URDF)
Before this commit: robot ymbot_d_description, 34 links, 33 joints
Joints:
- joint Right_Arm_Joint2: limit lower=-1.4 upper=0.03 effort=100 velocity=1 -> lower=-1.4 upper=0.2 effort=100 velocity=1
